File: coilcube/rev_c/coilcube.sch (EAGLE design)
At the start: 30 parts, among them J1 SCREW-TERMINAL_2_0.100, J3 EPIC-PROG-POGO-NO-LEGS, T1 NCHAN_MOSFET, T2 NCHAN_MOSFET, T3 NCHAN_MOSFET, U1 EPIC-CORE_A, U2 LTC3588_, U3 FM25LB

Commit message: preparing for a coilcube purchase
Parts:
- R4: DIGIKEY P4.7KGCT-ND -> RHM1.00MCFCT-ND
- R5: DIGIKEY P4.7KGCT-ND -> RHM4.7MCGDKR-ND
Changed lines of the file:
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@@
 <part name="GND4" library="supply1" deviceset="GND" device=""/>
 <part name="R4" library="rcl" deviceset="R-US_" device="R0603" value="1M">
-<attribute name="DIGIKEY" value="P4.7KGCT-ND"/>
+<attribute name="DIGIKEY" value="RHM1.00MCFCT-ND
+"/>
 </part>
 <part name="R5" library="rcl" deviceset="R-US_" device="R0603" value="4.7M">
-<attribute name="DIGIKEY" value="P4.7KGCT-ND"/>
+<attribute name="DIGIKEY" value="RHM4.7MCGDKR-ND
+"/>
 </part>
 </parts>
