File: hardware/epic2/rev_a/epic2.brd (EAGLE design)
At the start: 18 x 18 mm, 33 parts, among them J1 EPIC2-HEADER2, U1 RV-4162-C7, U2 FM25LBTDFN-8, U3 CC2538, X1 EPSON-FA-128, X3 ABS05-32.768KHZ-T

Commit message: no airwaires
Parts:
- removed C18: 10nF, passives:0402_CAP
- removed U1: RV-4162-C7, chips:MICRO-CRYSTAL-C7
- added C7: 10nF, passives:0402_CAP
- added R5, R7: 10k, passives:0402_RES
- added U5: RV-3049-C3, chips:MICRO-CRYSTAL-C3
- moved R1 5.35 mm to (10.3, 16.5)
- moved C10 2.21 mm to (3.96, 9.37)
- moved C14 1.93 mm to (4.70, 11.6)
- moved C6 1.89 mm to (4.70, 10.8)
- moved C13 0.87 mm to (16.2, 1.85), turned to 270 degrees
- moved C9 0.76 mm to (9.62, 14.1)
- moved R6 0.76 mm to (6.15, 1.85)
- moved C4 0.72 mm to (6.83, 12.7), turned to 180 degrees
- moved C15 0.68 mm to (17.0, 1.85)
- moved B1 0.25 mm to (5.36, 6.09)
- moved C11 0.25 mm to (6.15, 3.60)
- moved C12 0.25 mm to (6.93, 1.35)
- moved C16 0.25 mm to (7.72, 1.35)
- moved C3 0.25 mm to (6.93, 3.60)
- moved X3 0.25 mm to (8.97, 1.14)
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Connections:
- removed net RTC_CLKOUT: U1.2, U3.53
- new net !RTC_CS: U3.54, U5.8
- new net N$14: R7.2, U5.9
- new net N$16: R5.2, U5.1
- net !RTC_INT: now also U3.53, U5.7; no longer U1.6, U3.54
- net GND: now also C7.2, R5.1, R7.1, U5.6; no longer C18.2, U1.3
- net I2C_SCL: no longer U1.8
- net I2C_SDA: no longer U1.1
- net SPI_MISO: now also U5.5
- net SPI_MOSI: now also U5.10
- net SPI_SCK: now also U5.4
- net VCC: now also C7.1, U5.2; no longer C18.1, U1.5
Routing:
- net RTC_CLKOUT: track 22.6 -> 0.00 mm, vias 2 -> 0
- net N$15: track 4.18 -> 23.2 mm, vias 0 -> 2
- net !RTC_CS: track 0.00 -> 17.4 mm, vias 0 -> 2
- net SPI_MOSI: track 19.4 -> 29.0 mm, vias 1 -> 2
- net I2C_SCL: track 13.7 -> 4.50 mm, vias 2 -> 1
- net SPI_MISO: track 26.0 -> 34.5 mm, vias 1 -> 2
- net I2C_SDA: track 14.6 -> 6.87 mm, vias 2 -> 1
- net SPI_SCK: track 18.5 -> 26.0 mm, vias 1 -> 2
- net !RESET: track 8.10 -> 1.61 mm, vias 1 -> 0
- net VCC: track 29.6 -> 34.8 mm, vias 8 -> 11
- net N$1: track 2.62 -> 7.36 mm, vias 0 -> 2
- net GND: track 11.7 -> 15.9 mm, vias 33 -> 35
- net ANTENNA: track 0.00 -> 3.47 mm
- net ADC5: track 10.8 -> 8.31 mm, vias 0 -> 1
- net ADC4: track 10.1 -> 7.64 mm, vias 0 -> 1
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- removed copper zone on layer 1, net ANTENNA
- removed copper zone on layer 1, net RF_N
- removed copper zone on layer 1, net RF_P
Other:
- board size 18 x 18 mm -> 18.8 x 19.6 mm

Commit message: epic2: cleaned up a couple things
Parts:
- moved U$1 10.8 mm to (5.38, 1.22), turned to 90 degrees
- moved R5 0.61 mm to (16.8, 15.3)
Routing:
- net SPI_MISO: track 34.5 -> 35.5 mm
Changed lines of the file:
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@@
 <wire x1="17.9578" y1="17.9578" x2="0" y2="17.9578" width="0" layer="20"/>
 <wire x1="0" y1="17.9578" x2="0" y2="0" width="0" layer="20"/>
-<text x="4.4704" y="-1.7272" size="0.762" layer="21" font="vector" ratio="12" align="center-left">BC</text>
 <wire x1="0" y1="-0.8382" x2="0" y2="18.796" width="0" layer="46"/>
 <wire x1="0" y1="18.796" x2="18.796" y2="18.796" width="0" layer="46"/>
 <wire x1="18.796" y1="18.796" x2="18.796" y2="-0.8382" width="0" layer="46"/>
 <wire x1="18.796" y1="-0.8382" x2="0" y2="-0.8382" width="0" layer="46"/>
+<text x="17.5006" y="16.9926" size="0.762" layer="21" font="vector" ratio="12" rot="R90" align="bottom-center">BC</text>
 </plain>
 <attributes>
@@
 </autorouter>
 <elements>
-<element name="U$1" library="logos" package="UMICH_SOLID_75MIL" value="UMICH_SOLID_SMALL" x="-3.048" y="7.9756"/>
+<element name="U$1" library="logos" package="UMICH_SOLID_75MIL" value="UMICH_SOLID_SMALL" x="5.3848" y="1.2192" rot="R90"/>
 <element name="U2" library="chips" package="TDFN-8" value="FM25LBTDFN-8" x="5.7224" y="15.469" smashed="yes" rot="R270">
 <attribute name="DIGIKEY" value="FM25L04B-DGRA-ND" x="5.7224" y="15.469" size="1.778" layer="27" rot="R270" display="off"/>
@@
 <element name="C20" library="rcl" package="C0201" value="0.1uF" x="17.526" y="8.6614" rot="R90"/>
 <element name="U5" library="chips" package="MICRO-CRYSTAL-C3" value="RV-3049-C3" x="14.1986" y="15.2908" rot="R180"/>
-<element name="R5" library="passives" package="0402_RES" value="10k" x="16.8148" y="15.9004" rot="R90"/>
+<element name="R5" library="passives" package="0402_RES" value="10k" x="16.8148" y="15.2908" rot="R90"/>
 <element name="R7" library="passives" package="0402_RES" value="10k" x="14.9098" y="13.335" rot="R180"/>
 <element name="C7" library="passives" package="0402_CAP" value="10nF" x="14.5796" y="17.2466" rot="R180"/>
@@
 <contactref element="J1" pad="32"/>
 <via x="10.9474" y="1.016" extent="1-16" drill="0.2032"/>
-<wire x1="10.2108" y1="1.57606875" x2="10.79626875" y2="1.1938" width="0.1524" layer="1"/>
-<wire x1="10.79626875" y1="1.1938" x2="10.9474" y2="1.016" width="0.1524" layer="1"/>
 <via x="15.621" y="11.8872" extent="1-16" drill="0.2032"/>
 <via x="16.918940625" y="9.1948" extent="1-16" drill="0.2032"/>
@@
 <wire x1="3.52933125" y1="9.3726" x2="3.52933125" y2="9.17066875" width="0.1524" layer="1"/>
 <wire x1="3.52933125" y1="9.17066875" x2="4.318" y2="8.382" width="0.1524" layer="1"/>
-<via x="9.4742" y="15.7988" extent="1-16" drill="0.2032"/>
-<via x="11.4046" y="14.5034" extent="1-16" drill="0.2032"/>
+<via x="9.525" y="16.2306" extent="1-16" drill="0.2032"/>
+<via x="11.43" y="14.0716" extent="1-16" drill="0.2032"/>
 <wire x1="15.34286875" y1="13.335" x2="15.8496" y2="13.335" width="0.1524" layer="1"/>
 <wire x1="15.8496" y1="13.335" x2="16.8148" y2="14.3002" width="0.1524" layer="1"/>
-<wire x1="16.8148" y1="14.3002" x2="16.8148" y2="15.46733125" width="0.1524" layer="1"/>
-<wire x1="15.621" y1="11.8872" x2="16.23186875" y2="12.49806875" width="0.1524" layer="1"/>
+<wire x1="16.8148" y1="14.3002" x2="16.8148" y2="14.85773125" width="0.1524" layer="1"/>
 <wire x1="16.23186875" y1="12.49806875" x2="16.3576" y2="12.49806875" width="0.1524" layer="1"/>
 <wire x1="5.3594" y1="5.193459375" x2="5.461" y2="5.091859375" width="0.1524" layer="1"/>
@@
 <wire x1="6.9342" y1="0.91313125" x2="6.6548" y2="0.91313125" width="0.1524" layer="1"/>
 <wire x1="6.6548" y1="0.91313125" x2="6.1468" y2="1.42113125" width="0.1524" layer="1"/>
+<wire x1="10.9474" y1="1.016" x2="10.38733125" y2="1.57606875" width="0.1524" layer="1"/>
+<wire x1="10.38733125" y1="1.57606875" x2="10.2108" y2="1.57606875" width="0.1524" layer="1"/>
+<wire x1="15.621" y1="11.8872" x2="15.621" y2="12.0396" width="0.254" layer="1"/>
+<wire x1="15.621" y1="12.0396" x2="16.07946875" y2="12.49806875" width="0.254" layer="1"/>
+<wire x1="16.07946875" y1="12.49806875" x2="16.3576" y2="12.49806875" width="0.254" layer="1"/>
 </signal>
 <signal name="VCC">
@@
 <wire x1="15.4432" y1="2.1336" x2="16.02613125" y2="2.1336" width="0.1524" layer="1"/>
 <wire x1="16.02613125" y1="2.1336" x2="16.1798" y2="2.28726875" width="0.1524" layer="1"/>
-<via x="16.3322" y="17.1958" extent="1-16" drill="0.2032"/>
+<via x="16.2052" y="17.1196" extent="1-16" drill="0.2032"/>
 <wire x1="15.01266875" y1="17.2466" x2="15.06346875" y2="17.1958" width="0.1524" layer="1"/>
-<wire x1="15.06346875" y1="17.1958" x2="16.3322" y2="17.1958" width="0.1524" layer="1"/>
 <via x="5.969" y="10.7188" extent="1-16" drill="0.2032"/>
 <wire x1="5.969" y1="10.7188" x2="5.8928" y2="10.795" width="0.1524" layer="1"/>
 <wire x1="5.8928" y1="10.795" x2="5.13206875" y2="10.795" width="0.1524" layer="1"/>
+<wire x1="16.2052" y1="17.1196" x2="15.13966875" y2="17.1196" width="0.1524" layer="1"/>
+<wire x1="15.13966875" y1="17.1196" x2="15.01266875" y2="17.2466" width="0.1524" layer="1"/>
 </signal>
 <signal name="TCK">
@@
 <contactref element="J1" pad="24"/>
 <via x="14.6812" y="12.5222" extent="1-16" drill="0.2032"/>
-<wire x1="15.0368" y1="16.7157" x2="16.4789" y2="18.1578" width="0.1524" layer="15"/>
 <wire x1="14.18" y1="11.1696" x2="14.18" y2="12.021" width="0.1524" layer="1"/>
 <wire x1="14.18" y1="12.021" x2="14.6812" y2="12.5222" width="0.1524" layer="1"/>
 <wire x1="14.6812" y1="12.5222" x2="15.0368" y2="12.8778" width="0.1524" layer="15"/>
-<wire x1="15.0368" y1="12.8778" x2="15.0368" y2="16.7157" width="0.1524" layer="15"/>
+<wire x1="15.0368" y1="12.8778" x2="15.0368" y2="17.1958" width="0.1524" layer="15"/>
+<wire x1="15.0368" y1="17.1958" x2="15.3162" y2="17.4752" width="0.1524" layer="15"/>
+<wire x1="15.3162" y1="17.4752" x2="15.7963" y2="17.4752" width="0.1524" layer="15"/>
+<wire x1="15.7963" y1="17.4752" x2="16.4789" y2="18.1578" width="0.1524" layer="15"/>
 </signal>
 <signal name="BOOTLOADER_CTRL">
@@
 <via x="12.827" y="15.494" extent="1-16" drill="0.2032"/>
 <wire x1="9.017" y1="12.8778" x2="9.017" y2="13.97" width="0.1524" layer="15"/>
-<wire x1="12.827" y1="15.494" x2="9.9314" y2="15.494" width="0.1524" layer="16"/>
-<wire x1="9.9314" y1="15.494" x2="8.9408" y2="14.5034" width="0.1524" layer="16"/>
-<wire x1="8.9408" y1="14.5034" x2="8.4836" y2="14.5034" width="0.1524" layer="16"/>
+<wire x1="12.827" y1="15.494" x2="9.9822" y2="15.494" width="0.1524" layer="16"/>
+<wire x1="9.9822" y1="15.494" x2="8.9916" y2="14.5034" width="0.1524" layer="16"/>
+<wire x1="8.9916" y1="14.5034" x2="8.4836" y2="14.5034" width="0.1524" layer="16"/>
 <wire x1="16.1036" y1="9.8298" x2="14.4018" y2="11.5316" width="0.1524" layer="15"/>
 <wire x1="14.4018" y1="11.5316" x2="10.3632" y2="11.5316" width="0.1524" layer="15"/>
@@
 <contactref element="R2" pad="1"/>
 <wire x1="1.70053125" y1="17.12086875" x2="1.651" y2="17.1704" width="0.1524" layer="1"/>
-<wire x1="2.413" y1="15.59686875" x2="2.413" y2="16.4084" width="0.1524" layer="1"/>
-<wire x1="2.413" y1="16.4084" x2="1.651" y2="17.1704" width="0.1524" layer="1"/>
+<wire x1="1.651" y1="17.1704" x2="2.1336" y2="16.6878" width="0.1524" layer="1"/>
+<wire x1="2.1336" y1="16.6878" x2="2.1336" y2="15.87626875" width="0.1524" layer="1"/>
+<wire x1="2.1336" y1="15.87626875" x2="2.413" y2="15.59686875" width="0.1524" layer="1"/>
 </signal>
 <signal name="N$11">
@@
 <contactref element="U3" pad="5"/>
 <contactref element="J1" pad="14"/>
-<via x="2.9464" y="16.4338" extent="1-16" drill="0.2032"/>
+<via x="2.8448" y="16.3322" extent="1-16" drill="0.2032"/>
 <wire x1="15.494" y1="9.525" x2="15.494" y2="6.7818" width="0.1524" layer="15"/>
 <wire x1="15.494" y1="6.7818" x2="16.8731" y2="5.4027" width="0.1524" layer="15"/>
@@
 <wire x1="12.5646" y1="16.3068" x2="11.9126" y2="16.3068" width="0.1524" layer="1"/>
 <wire x1="11.9126" y1="16.3068" x2="11.8872" y2="16.3322" width="0.1524" layer="1"/>
-<wire x1="3.048" y1="16.3322" x2="11.8872" y2="16.3322" width="0.1524" layer="16"/>
-<wire x1="3.7724" y1="15.944" x2="3.4362" y2="15.944" width="0.1524" layer="1"/>
-<wire x1="3.4362" y1="15.944" x2="2.9464" y2="16.4338" width="0.1524" layer="1"/>
-<wire x1="3.048" y1="16.3322" x2="2.9464" y2="16.4338" width="0.1524" layer="16"/>
+<wire x1="3.7724" y1="15.944" x2="3.233" y2="15.944" width="0.1524" layer="1"/>
+<wire x1="3.048" y1="16.3322" x2="2.8448" y2="16.3322" width="0.1524" layer="16"/>
 <wire x1="9.906" y1="10.922" x2="4.3942" y2="16.4338" width="0.1524" layer="15"/>
-<wire x1="4.3942" y1="16.4338" x2="2.9464" y2="16.4338" width="0.1524" layer="15"/>
+<wire x1="4.3942" y1="16.4338" x2="2.8448" y2="16.3322" width="0.1524" layer="15"/>
 <wire x1="16.8731" y1="5.4027" x2="18.0816" y2="5.4027" width="0.1524" layer="15"/>
 <wire x1="18.0816" y1="5.4027" x2="18.1578" y2="5.4789" width="0.1524" layer="15"/>
+<wire x1="11.8872" y1="16.3322" x2="11.3538" y2="15.7988" width="0.1524" layer="16"/>
+<wire x1="11.3538" y1="15.7988" x2="9.8552" y2="15.7988" width="0.1524" layer="16"/>
+<wire x1="9.8552" y1="15.7988" x2="9.5758" y2="15.5194" width="0.1524" layer="16"/>
+<wire x1="9.5758" y1="15.5194" x2="3.8608" y2="15.5194" width="0.1524" layer="16"/>
+<wire x1="3.8608" y1="15.5194" x2="2.8448" y2="16.3322" width="0.1524" layer="16"/>
+<wire x1="3.233" y1="15.944" x2="2.8448" y2="16.3322" width="0.1524" layer="1"/>
 </signal>
 <signal name="N$13">
@@
 <contactref element="R5" pad="2"/>
 <wire x1="15.7986" y1="16.3408" x2="15.86766875" y2="16.3408" width="0.1524" layer="1"/>
-<wire x1="15.86766875" y1="16.3408" x2="16.8148" y2="16.33346875" width="0.1524" layer="1"/>
+<wire x1="16.8148" y1="15.72386875" x2="16.41553125" y2="15.72386875" width="0.1524" layer="1"/>
+<wire x1="16.41553125" y1="15.72386875" x2="15.7986" y2="16.3408" width="0.1524" layer="1"/>
 </signal>
 <signal name="!RTC_CS">

Commit message: updates to epic2 brd
Parts:
- moved R2 0.76 mm to (2.41, 15.9)
Routing:
- net LED_RED: track 8.83 -> 9.61 mm
- net N$7: track 1.96 -> 1.35 mm
Changed lines of the file:
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@@
 <layer number="13" name="Route13" color="4" fill="5" visible="no" active="no"/>
 <layer number="14" name="Route14" color="1" fill="6" visible="no" active="no"/>
-<layer number="15" name="Route15" color="3" fill="6" visible="no" active="yes"/>
-<layer number="16" name="Bottom" color="1" fill="1" visible="no" active="yes"/>
+<layer number="15" name="Route15" color="3" fill="6" visible="yes" active="yes"/>
+<layer number="16" name="Bottom" color="1" fill="1" visible="yes" active="yes"/>
 <layer number="17" name="Pads" color="2" fill="1" visible="yes" active="yes"/>
 <layer number="18" name="Vias" color="2" fill="1" visible="yes" active="yes"/>
@@
 <attribute name="NAME" x="0.3192" y="16.7386" size="1.016" layer="25" font="vector" ratio="12" rot="R90" align="bottom-center"/>
 </element>
-<element name="R2" library="passives" package="0402_RES" value="1k" x="2.413" y="15.1638" rot="R270"/>
+<element name="R2" library="passives" package="0402_RES" value="1k" x="2.413" y="15.9258" rot="R270"/>
 <element name="R3" library="passives" package="0402_RES" value="1k" x="0.8382" y="15.1892" rot="R270"/>
 <element name="R4" library="passives" package="0402_RES" value="1k" x="1.6256" y="15.1638" rot="R270"/>
@@
 <contactref element="D1" pad="2"/>
 <contactref element="R2" pad="1"/>
-<wire x1="1.70053125" y1="17.12086875" x2="1.651" y2="17.1704" width="0.1524" layer="1"/>
-<wire x1="1.651" y1="17.1704" x2="2.1336" y2="16.6878" width="0.1524" layer="1"/>
-<wire x1="2.1336" y1="16.6878" x2="2.1336" y2="15.87626875" width="0.1524" layer="1"/>
-<wire x1="2.1336" y1="15.87626875" x2="2.413" y2="15.59686875" width="0.1524" layer="1"/>
+<wire x1="2.413" y1="16.35886875" x2="2.413" y2="16.7894" width="0.1524" layer="1"/>
+<wire x1="2.413" y1="16.7894" x2="2.032" y2="17.1704" width="0.1524" layer="1"/>
+<wire x1="2.032" y1="17.1704" x2="1.651" y2="17.1704" width="0.1524" layer="1"/>
 </signal>
 <signal name="N$11">
@@
 <contactref element="U3" pad="29"/>
 <via x="8.001" y="10.9474" extent="1-16" drill="0.2032"/>
-<via x="2.8956" y="13.97" extent="1-16" drill="0.2032"/>
+<via x="2.8956" y="13.8176" extent="1-16" drill="0.2032"/>
 <wire x1="7.855" y1="10.3446" x2="7.855" y2="10.8014" width="0.1524" layer="1"/>
 <wire x1="7.855" y1="10.8014" x2="8.001" y2="10.9474" width="0.1524" layer="1"/>
 <wire x1="8.001" y1="10.9474" x2="7.5438" y2="11.4046" width="0.1524" layer="15"/>
-<wire x1="6.3754" y1="13.7922" x2="3.0734" y2="13.7922" width="0.1524" layer="15"/>
-<wire x1="3.0734" y1="13.7922" x2="2.8956" y2="13.97" width="0.1524" layer="15"/>
-<wire x1="2.413" y1="14.73073125" x2="2.64286875" y2="14.73073125" width="0.1524" layer="1"/>
-<wire x1="2.64286875" y1="14.73073125" x2="2.8956" y2="14.478" width="0.1524" layer="1"/>
-<wire x1="2.8956" y1="14.478" x2="2.8956" y2="13.97" width="0.1524" layer="1"/>
 <wire x1="7.5438" y1="11.4046" x2="7.5438" y2="12.6238" width="0.1524" layer="15"/>
 <wire x1="7.5438" y1="12.6238" x2="6.3754" y2="13.7922" width="0.1524" layer="15"/>
+<wire x1="2.3368" y1="14.5542" x2="2.8956" y2="13.9954" width="0.1524" layer="1"/>
+<wire x1="2.8956" y1="13.9954" x2="2.8956" y2="13.8176" width="0.1524" layer="1"/>
+<wire x1="6.3754" y1="13.7922" x2="2.921" y2="13.7922" width="0.1524" layer="15"/>
+<wire x1="2.921" y1="13.7922" x2="2.8956" y2="13.8176" width="0.1524" layer="15"/>
+<wire x1="2.3368" y1="14.5542" x2="2.3368" y2="15.41653125" width="0.1524" layer="1"/>
+<wire x1="2.3368" y1="15.41653125" x2="2.413" y2="15.49273125" width="0.1524" layer="1"/>
 </signal>
 <signal name="ADC5">
@@
 <contactref element="U3" pad="5"/>
 <contactref element="J1" pad="14"/>
-<via x="2.8448" y="16.3322" extent="1-16" drill="0.2032"/>
+<via x="2.8956" y="14.7574" extent="1-16" drill="0.2032"/>
 <wire x1="15.494" y1="9.525" x2="15.494" y2="6.7818" width="0.1524" layer="15"/>
 <wire x1="15.494" y1="6.7818" x2="16.8731" y2="5.4027" width="0.1524" layer="15"/>
@@
 <wire x1="12.5646" y1="16.3068" x2="11.9126" y2="16.3068" width="0.1524" layer="1"/>
 <wire x1="11.9126" y1="16.3068" x2="11.8872" y2="16.3322" width="0.1524" layer="1"/>
-<wire x1="3.7724" y1="15.944" x2="3.233" y2="15.944" width="0.1524" layer="1"/>
-<wire x1="3.048" y1="16.3322" x2="2.8448" y2="16.3322" width="0.1524" layer="16"/>
-<wire x1="9.906" y1="10.922" x2="4.3942" y2="16.4338" width="0.1524" layer="15"/>
-<wire x1="4.3942" y1="16.4338" x2="2.8448" y2="16.3322" width="0.1524" layer="15"/>
 <wire x1="16.8731" y1="5.4027" x2="18.0816" y2="5.4027" width="0.1524" layer="15"/>
 <wire x1="18.0816" y1="5.4027" x2="18.1578" y2="5.4789" width="0.1524" layer="15"/>
 <wire x1="11.8872" y1="16.3322" x2="11.3538" y2="15.7988" width="0.1524" layer="16"/>
 <wire x1="11.3538" y1="15.7988" x2="9.8552" y2="15.7988" width="0.1524" layer="16"/>
-<wire x1="9.8552" y1="15.7988" x2="9.5758" y2="15.5194" width="0.1524" layer="16"/>
-<wire x1="9.5758" y1="15.5194" x2="3.8608" y2="15.5194" width="0.1524" layer="16"/>
-<wire x1="3.8608" y1="15.5194" x2="2.8448" y2="16.3322" width="0.1524" layer="16"/>
-<wire x1="3.233" y1="15.944" x2="2.8448" y2="16.3322" width="0.1524" layer="1"/>
+<wire x1="9.8552" y1="15.7988" x2="9.0932" y2="15.0368" width="0.1524" layer="16"/>
+<wire x1="9.0932" y1="15.0368" x2="8.2296" y2="15.0368" width="0.1524" layer="16"/>
+<wire x1="8.2296" y1="15.0368" x2="7.9502" y2="14.7574" width="0.1524" layer="16"/>
+<wire x1="7.9502" y1="14.7574" x2="2.8956" y2="14.7574" width="0.1524" layer="16"/>
+<wire x1="3.7724" y1="15.944" x2="3.4726" y2="15.944" width="0.1524" layer="1"/>
+<wire x1="3.4726" y1="15.944" x2="2.8956" y2="15.367" width="0.1524" layer="1"/>
+<wire x1="2.8956" y1="15.367" x2="2.8956" y2="14.7574" width="0.1524" layer="1"/>
+<wire x1="9.906" y1="10.922" x2="6.0706" y2="14.7574" width="0.1524" layer="15"/>
+<wire x1="6.0706" y1="14.7574" x2="2.8956" y2="14.7574" width="0.1524" layer="15"/>
 </signal>
 <signal name="N$13">
