File: hardware/bigben/rev_a/bigben.sch (EAGLE design)
At the start: 13 parts, among them J3 IMPULSE_GECKO_HEADER, U1 RV-3049-C3, U2 FM25LBTDFN-8

Commit message: shipped bigben
Parts:
- removed R5, R6: 10k, passives:RESISTOR
- R3, R4: value 4.7k -> 10k
- U2: value FM25LBTDFN-8 -> FM25V20-DG; device chips:FM25LBTDFN-8 -> chips:FM25V20-DG; MOUSER 877-FM25V20-DG -> (none)
Connections:
- removed net !FRAM_HOLD: R2.1, U2.!HOLD
- removed net !FRAM_WP: R3.1, U2.!WP
- net GND: now also R2.1, R3.1; no longer R5.1, R6.1
- net N$6: now also R4.2; no longer R6.2
- net N$7: now also R3.2; no longer R5.2
- net RTC_CS: now also R2.2; no longer R4.2
- net VCC: now also U2.!HOLD, U2.!WP; no longer R2.2, R3.2
Other:
- moved on the sheet: R2, R3, R4
Changed lines of the file:
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@@
 <part name="GND1" library="supply1" deviceset="GND" device=""/>
 <part name="P+2" library="supply1" deviceset="VCC" device=""/>
-<part name="U2" library="chips" deviceset="FM25LB" device="TDFN-8">
-<attribute name="MOUSER" value="877-FM25V20-DG"/>
-</part>
 <part name="GND9" library="supply1" deviceset="GND" device=""/>
 <part name="P+5" library="supply1" deviceset="VCC" device=""/>
 <part name="R1" library="passives" deviceset="RESISTOR" device="" value="4.7k"/>
-<part name="R2" library="passives" deviceset="RESISTOR" device="" value="4.7k"/>
-<part name="R3" library="passives" deviceset="RESISTOR" device="" value="4.7k"/>
 <part name="P+7" library="supply1" deviceset="VCC" device=""/>
 <part name="C2" library="passives" deviceset="CAPACITOR" device="" value="0.1uF"/>
@@
 <part name="GND13" library="supply1" deviceset="GND" device=""/>
 <part name="GND14" library="supply1" deviceset="GND" device=""/>
-<part name="R6" library="passives" deviceset="RESISTOR" device="" value="10k"/>
-<part name="R5" library="passives" deviceset="RESISTOR" device="" value="10k"/>
+<part name="R4" library="passives" deviceset="RESISTOR" device="" value="10k"/>
+<part name="R3" library="passives" deviceset="RESISTOR" device="" value="10k"/>
 <part name="C1" library="passives" deviceset="CAPACITOR" device="" value="10nF"/>
-<part name="R4" library="passives" deviceset="RESISTOR" device="" value="4.7k"/>
+<part name="R2" library="passives" deviceset="RESISTOR" device="" value="4.7k"/>
 <part name="GND11" library="supply1" deviceset="GND" device=""/>
 <part name="GND12" library="supply1" deviceset="GND" device=""/>
 <part name="LOGO1" library="logos" deviceset="UMICH_SOLID" device="_TINY"/>
+<part name="U2" library="chips" deviceset="FM25" device="V20-DG"/>
+<part name="P+1" library="supply1" deviceset="VCC" device=""/>
 </parts>
 <sheets>
@@
 <instance part="GND13" gate="1" x="165.1" y="55.88"/>
 <instance part="GND14" gate="1" x="193.04" y="48.26"/>
-<instance part="R6" gate="G$1" x="165.1" y="73.66" smashed="yes" rot="R90">
+<instance part="R4" gate="G$1" x="165.1" y="73.66" smashed="yes" rot="R90">
 <attribute name="NAME" x="163.6014" y="69.85" size="1.778" layer="95" rot="R90"/>
 <attribute name="VALUE" x="168.402" y="69.85" size="1.778" layer="96" rot="R90"/>
 </instance>
-<instance part="R5" gate="G$1" x="193.04" y="58.42" smashed="yes" rot="R90">
+<instance part="R3" gate="G$1" x="193.04" y="58.42" smashed="yes" rot="R90">
 <attribute name="NAME" x="191.5414" y="54.61" size="1.778" layer="95" rot="R90"/>
 <attribute name="VALUE" x="196.342" y="54.61" size="1.778" layer="96" rot="R90"/>
 </instance>
 <instance part="C1" gate="G$1" x="154.94" y="73.66"/>
-<instance part="U2" gate="G$1" x="53.34" y="60.96">
-<attribute name="MOUSER" x="53.34" y="60.96" size="1.27" layer="96" display="off"/>
-</instance>
 <instance part="GND9" gate="1" x="38.1" y="43.18"/>
 <instance part="P+5" gate="VCC" x="38.1" y="73.66"/>
 <instance part="R1" gate="G$1" x="81.28" y="66.04" rot="R90"/>
-<instance part="R2" gate="G$1" x="91.44" y="66.04" rot="R90"/>
-<instance part="R3" gate="G$1" x="101.6" y="66.04" rot="R90"/>
 <instance part="P+7" gate="VCC" x="91.44" y="81.28"/>
 <instance part="C2" gate="G$1" x="35.56" y="63.5"/>
-<instance part="R4" gate="G$1" x="203.2" y="66.04" smashed="yes" rot="R90">
+<instance part="R2" gate="G$1" x="203.2" y="66.04" smashed="yes" rot="R90">
 <attribute name="NAME" x="201.7014" y="62.23" size="1.778" layer="95" rot="R90"/>
 <attribute name="VALUE" x="206.502" y="62.23" size="1.778" layer="96" rot="R90"/>
@@
 <instance part="GND12" gate="1" x="172.72" y="134.62"/>
 <instance part="LOGO1" gate="G$1" x="233.172" y="173.99"/>
+<instance part="U2" gate="G$1" x="53.34" y="60.96"/>
+<instance part="P+1" gate="VCC" x="81.28" y="81.28"/>
 </instances>
 <busses>
@@
 <wire x1="165.1" y1="60.96" x2="165.1" y2="58.42" width="0.1524" layer="91"/>
 <pinref part="GND13" gate="1" pin="GND"/>
-<pinref part="R6" gate="G$1" pin="1"/>
+<pinref part="R4" gate="G$1" pin="1"/>
 <wire x1="165.1" y1="68.58" x2="165.1" y2="60.96" width="0.1524" layer="91"/>
 <junction x="165.1" y="60.96"/>
@@
 </segment>
 <segment>
-<pinref part="R5" gate="G$1" pin="1"/>
+<pinref part="R3" gate="G$1" pin="1"/>
 <pinref part="GND14" gate="1" pin="GND"/>
 <wire x1="193.04" y1="50.8" x2="193.04" y2="53.34" width="0.1524" layer="91"/>
 </segment>
 <segment>
-<pinref part="U2" gate="G$1" pin="VSS"/>
 <wire x1="40.64" y1="55.88" x2="38.1" y2="55.88" width="0.1524" layer="91"/>
 <wire x1="38.1" y1="55.88" x2="35.56" y2="55.88" width="0.1524" layer="91"/>
@@
 <junction x="38.1" y="55.88"/>
 <pinref part="C2" gate="G$1" pin="2"/>
-</segment>
-<segment>
-<pinref part="R4" gate="G$1" pin="1"/>
+<pinref part="U2" gate="G$1" pin="VSS"/>
+</segment>
+<segment>
+<pinref part="R2" gate="G$1" pin="1"/>
 <wire x1="203.2" y1="60.96" x2="203.2" y2="50.8" width="0.1524" layer="91"/>
 <pinref part="GND11" gate="1" pin="GND"/>
@@
 </segment>
 <segment>
-<pinref part="U2" gate="G$1" pin="VDD"/>
 <wire x1="35.56" y1="66.04" x2="35.56" y2="68.58" width="0.1524" layer="91"/>
 <wire x1="35.56" y1="68.58" x2="38.1" y2="68.58" width="0.1524" layer="91"/>
@@
 <pinref part="P+5" gate="VCC" pin="VCC"/>
 <pinref part="C2" gate="G$1" pin="1"/>
-</segment>
-<segment>
+<pinref part="U2" gate="G$1" pin="VDD"/>
+</segment>
+<segment>
+<pinref part="P+1" gate="VCC" pin="VCC"/>
 <pinref part="R1" gate="G$1" pin="2"/>
-<wire x1="81.28" y1="71.12" x2="81.28" y2="76.2" width="0.1524" layer="91"/>
+<wire x1="81.28" y1="71.12" x2="81.28" y2="78.74" width="0.1524" layer="91"/>
+</segment>
+<segment>
 <pinref part="P+7" gate="VCC" pin="VCC"/>
-<wire x1="81.28" y1="76.2" x2="91.44" y2="76.2" width="0.1524" layer="91"/>
-<wire x1="91.44" y1="76.2" x2="91.44" y2="78.74" width="0.1524" layer="91"/>
-<pinref part="R2" gate="G$1" pin="2"/>
-<wire x1="91.44" y1="76.2" x2="91.44" y2="71.12" width="0.1524" layer="91"/>
-<junction x="91.44" y="76.2"/>
-<wire x1="91.44" y1="76.2" x2="101.6" y2="76.2" width="0.1524" layer="91"/>
-<pinref part="R3" gate="G$1" pin="2"/>
-<wire x1="101.6" y1="76.2" x2="101.6" y2="71.12" width="0.1524" layer="91"/>
+<wire x1="66.04" y1="53.34" x2="68.58" y2="53.34" width="0.1524" layer="91"/>
+<pinref part="U2" gate="G$1" pin="!HOLD"/>
+<wire x1="68.58" y1="53.34" x2="91.44" y2="53.34" width="0.1524" layer="91"/>
+<wire x1="91.44" y1="53.34" x2="91.44" y2="78.74" width="0.1524" layer="91"/>
+<wire x1="66.04" y1="50.8" x2="68.58" y2="50.8" width="0.1524" layer="91"/>
+<pinref part="U2" gate="G$1" pin="!WP"/>
+<wire x1="68.58" y1="50.8" x2="68.58" y2="53.34" width="0.1524" layer="91"/>
+<junction x="68.58" y="53.34"/>
 </segment>
 </net>
@@
 </segment>
 <segment>
-<pinref part="U2" gate="G$1" pin="!CS"/>
 <pinref part="R1" gate="G$1" pin="1"/>
 <wire x1="66.04" y1="58.42" x2="81.28" y2="58.42" width="0.1524" layer="91"/>
@@
 <wire x1="86.36" y1="58.42" x2="86.36" y2="60.96" width="0.1524" layer="91"/>
 <label x="86.36" y="60.96" size="1.27" layer="95" rot="R90" xref="yes"/>
-</segment>
-</net>
-<net name="!FRAM_HOLD" class="0">
-<segment>
-<pinref part="U2" gate="G$1" pin="!HOLD"/>
-<pinref part="R2" gate="G$1" pin="1"/>
-<wire x1="66.04" y1="53.34" x2="91.44" y2="53.34" width="0.1524" layer="91"/>
-<wire x1="91.44" y1="53.34" x2="91.44" y2="60.96" width="0.1524" layer="91"/>
-</segment>
-</net>
-<net name="!FRAM_WP" class="0">
-<segment>
-<pinref part="U2" gate="G$1" pin="!WP"/>
-<pinref part="R3" gate="G$1" pin="1"/>
-<wire x1="66.04" y1="50.8" x2="101.6" y2="50.8" width="0.1524" layer="91"/>
-<wire x1="101.6" y1="50.8" x2="101.6" y2="60.96" width="0.1524" layer="91"/>
+<pinref part="U2" gate="G$1" pin="!CS"/>
 </segment>
 </net>
@@
 </segment>
 <segment>
-<pinref part="U2" gate="G$1" pin="SI"/>
 <wire x1="66.04" y1="66.04" x2="68.58" y2="66.04" width="0.1524" layer="91"/>
 <label x="68.58" y="66.04" size="1.27" layer="95" xref="yes"/>
+<pinref part="U2" gate="G$1" pin="SI"/>
 </segment>
 </net>
@@
 </segment>
 <segment>
-<pinref part="U2" gate="G$1" pin="SO"/>
 <wire x1="66.04" y1="63.5" x2="68.58" y2="63.5" width="0.1524" layer="91"/>
 <label x="68.58" y="63.5" size="1.27" layer="95" xref="yes"/>
+<pinref part="U2" gate="G$1" pin="SO"/>
 </segment>
 </net>
@@
 </segment>
 <segment>
-<pinref part="U2" gate="G$1" pin="SCK"/>
 <wire x1="66.04" y1="60.96" x2="68.58" y2="60.96" width="0.1524" layer="91"/>
 <label x="68.58" y="60.96" size="1.27" layer="95" xref="yes"/>
+<pinref part="U2" gate="G$1" pin="SCK"/>
 </segment>
 </net>
@@
 <wire x1="187.96" y1="73.66" x2="203.2" y2="73.66" width="0.1524" layer="91"/>
 <label x="208.28" y="73.66" size="1.27" layer="95" xref="yes"/>
-<pinref part="R4" gate="G$1" pin="2"/>
+<pinref part="R2" gate="G$1" pin="2"/>
 <wire x1="203.2" y1="73.66" x2="208.28" y2="73.66" width="0.1524" layer="91"/>
 <wire x1="203.2" y1="73.66" x2="203.2" y2="71.12" width="0.1524" layer="91"/>
@@
 <pinref part="U1" gate="G$1" pin="VBACKUP"/>
 <wire x1="167.64" y1="83.82" x2="165.1" y2="83.82" width="0.1524" layer="91"/>
-<pinref part="R6" gate="G$1" pin="2"/>
+<pinref part="R4" gate="G$1" pin="2"/>
 <wire x1="165.1" y1="83.82" x2="165.1" y2="78.74" width="0.1524" layer="91"/>
 </segment>
@@
 <segment>
 <pinref part="U1" gate="G$1" pin="CLKOE"/>
-<pinref part="R5" gate="G$1" pin="2"/>
+<pinref part="R3" gate="G$1" pin="2"/>
 <wire x1="187.96" y1="66.04" x2="193.04" y2="66.04" width="0.1524" layer="91"/>
 <wire x1="193.04" y1="66.04" x2="193.04" y2="63.5" width="0.1524" layer="91"/>

Commit message: bigben files updated with picture
Other:
- note added: "Battery"
- note added: "Impulse Connection"
- note added: "RTC"
- moved on the sheet: J3
Changed lines of the file:
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@@
 <sheet>
 <plain>
-<text x="53.34" y="76.2" size="2.54" layer="97">FRAM</text>
+<text x="53.34" y="76.2" size="2.54" layer="98" align="bottom-center">FRAM</text>
+<text x="55.88" y="162.56" size="2.54" layer="98" align="bottom-center">Impulse Connection</text>
+<text x="177.8" y="93.98" size="2.54" layer="98" align="bottom-center">RTC</text>
+<text x="165.1" y="152.4" size="2.54" layer="98" align="bottom-center">Battery</text>
 </plain>
 <instances>
-<instance part="GND1" gate="1" x="53.34" y="124.46"/>
-<instance part="P+2" gate="VCC" x="53.34" y="157.48"/>
+<instance part="GND1" gate="1" x="78.74" y="121.92"/>
+<instance part="P+2" gate="VCC" x="78.74" y="154.94"/>
 <instance part="FRAME1" gate="G$1" x="0" y="0"/>
 <instance part="FRAME1" gate="G$2" x="147.32" y="0"/>
-<instance part="J3" gate="G$1" x="27.94" y="144.78"/>
+<instance part="J3" gate="G$1" x="53.34" y="142.24"/>
 <instance part="U1" gate="G$1" x="177.8" y="73.66"/>
 <instance part="BT1" gate="G$1" x="157.48" y="142.24"/>
@@
 <net name="GND" class="0">
 <segment>
-<wire x1="38.1" y1="137.16" x2="53.34" y2="137.16" width="0.1524" layer="91"/>
+<wire x1="63.5" y1="134.62" x2="78.74" y2="134.62" width="0.1524" layer="91"/>
 <pinref part="GND1" gate="1" pin="GND"/>
-<wire x1="53.34" y1="137.16" x2="53.34" y2="127" width="0.1524" layer="91"/>
+<wire x1="78.74" y1="134.62" x2="78.74" y2="124.46" width="0.1524" layer="91"/>
 <pinref part="J3" gate="G$1" pin="GND"/>
 </segment>
@@
 <net name="VCC" class="0">
 <segment>
-<wire x1="38.1" y1="152.4" x2="53.34" y2="152.4" width="0.1524" layer="91"/>
+<wire x1="63.5" y1="149.86" x2="78.74" y2="149.86" width="0.1524" layer="91"/>
 <pinref part="P+2" gate="VCC" pin="VCC"/>
-<wire x1="53.34" y1="152.4" x2="53.34" y2="154.94" width="0.1524" layer="91"/>
+<wire x1="78.74" y1="149.86" x2="78.74" y2="152.4" width="0.1524" layer="91"/>
 <pinref part="J3" gate="G$1" pin="VREG"/>
 </segment>
@@
 <net name="!FRAM_CS" class="0">
 <segment>
-<label x="40.64" y="142.24" size="1.27" layer="95" xref="yes"/>
+<label x="66.04" y="139.7" size="1.27" layer="95" xref="yes"/>
 <pinref part="J3" gate="G$1" pin="TRIGGER/P2.1"/>
-<wire x1="40.64" y1="142.24" x2="38.1" y2="142.24" width="0.1524" layer="91"/>
+<wire x1="66.04" y1="139.7" x2="63.5" y2="139.7" width="0.1524" layer="91"/>
 </segment>
 <segment>
@@
 <net name="VCAP" class="0">
 <segment>
-<label x="40.64" y="154.94" size="1.27" layer="95" xref="yes"/>
+<label x="66.04" y="152.4" size="1.27" layer="95" xref="yes"/>
 <pinref part="J3" gate="G$1" pin="VCAP"/>
-<wire x1="40.64" y1="154.94" x2="38.1" y2="154.94" width="0.1524" layer="91"/>
+<wire x1="66.04" y1="152.4" x2="63.5" y2="152.4" width="0.1524" layer="91"/>
 </segment>
 </net>
 <net name="SHD" class="0">
 <segment>
-<label x="40.64" y="144.78" size="1.27" layer="95" xref="yes"/>
+<label x="66.04" y="142.24" size="1.27" layer="95" xref="yes"/>
 <pinref part="J3" gate="G$1" pin="SHTDWN/P2.0"/>
-<wire x1="40.64" y1="144.78" x2="38.1" y2="144.78" width="0.1524" layer="91"/>
+<wire x1="66.04" y1="142.24" x2="63.5" y2="142.24" width="0.1524" layer="91"/>
 </segment>
 </net>
@@
 <segment>
 <pinref part="J3" gate="G$1" pin="MOSI/SDA"/>
-<wire x1="38.1" y1="132.08" x2="40.64" y2="132.08" width="0.1524" layer="91"/>
-<label x="40.64" y="132.08" size="1.27" layer="95" xref="yes"/>
+<wire x1="63.5" y1="129.54" x2="66.04" y2="129.54" width="0.1524" layer="91"/>
+<label x="66.04" y="129.54" size="1.27" layer="95" xref="yes"/>
 </segment>
 <segment>
@@
 <segment>
 <pinref part="J3" gate="G$1" pin="MISO"/>
-<wire x1="38.1" y1="129.54" x2="40.64" y2="129.54" width="0.1524" layer="91"/>
-<label x="40.64" y="129.54" size="1.27" layer="95" xref="yes"/>
+<wire x1="63.5" y1="127" x2="66.04" y2="127" width="0.1524" layer="91"/>
+<label x="66.04" y="127" size="1.27" layer="95" xref="yes"/>
 </segment>
 <segment>
@@
 <segment>
 <pinref part="J3" gate="G$1" pin="SCL"/>
-<wire x1="38.1" y1="127" x2="40.64" y2="127" width="0.1524" layer="91"/>
-<label x="40.64" y="127" size="1.27" layer="95" xref="yes"/>
+<wire x1="63.5" y1="124.46" x2="66.04" y2="124.46" width="0.1524" layer="91"/>
+<label x="66.04" y="124.46" size="1.27" layer="95" xref="yes"/>
 </segment>
 <segment>
@@
 <segment>
 <pinref part="J3" gate="G$1" pin="OVRVLT/P1.7"/>
-<label x="40.64" y="147.32" size="1.27" layer="95" xref="yes"/>
-<wire x1="38.1" y1="147.32" x2="40.64" y2="147.32" width="0.1524" layer="91"/>
-</segment>
-</net>
+<label x="66.04" y="144.78" size="1.27" layer="95" xref="yes"/>
+<wire x1="63.5" y1="144.78" x2="66.04" y2="144.78" width="0.1524" layer="91"/>
+</segment>
+</net>
