File: hardware/blast/rev_a/blast.brd (EAGLE design)
At the start: 32.5 x 13 mm, 35 parts, among them J2 TC2030-CTX-NL, J3 IMPULSE_GECKO_HEADER, Q1 MOSFET-NCHANNELXFDN-3, U2 FM25LBTDFN-8, U3 NRF51822QF, X2 16MHz

Commit message: not sure what i changed
Parts:
- moved R8 15.3 mm to (11.9, 11.6), turned to 90 degrees
Changed lines of the file:
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@@
 <attribute name="VALUE" x="10.0973875" y="9.236328125" size="1.016" layer="27" font="vector" ratio="12" rot="R180" align="bottom-center"/>
 </element>
-<element name="R8" library="passives" package="0402_RES" value="12k" x="23.368" y="1.524">
-<attribute name="DIGIKEY" value="RHM12.0KCDCT-ND" x="23.368" y="1.524" size="1.778" layer="27" display="off"/>
+<element name="R8" library="passives" package="0402_RES" value="12k" x="11.938" y="11.6332" rot="R90">
+<attribute name="DIGIKEY" value="RHM12.0KCDCT-ND" x="11.938" y="11.6332" size="1.778" layer="27" rot="R90" display="off"/>
 </element>
 <element name="J3" library="gecko" package="HEADER1X9/0.05IN" value="IMPULSE_GECKO_HEADER" x="31.369" y="6.477" rot="R90"/>
@@
 <contactref element="U3" pad="24"/>
 <contactref element="R8" pad="1"/>
-<wire x1="12.3808" y1="10.2326" x2="22.93493125" y2="1.524" width="0" layer="19" extent="1-1"/>
+<wire x1="12.3808" y1="10.2326" x2="11.938" y2="11.20013125" width="0" layer="19" extent="1-1"/>
 </signal>
 <signal name="SWDIO">
