File: hardware/blast/rev_a/blast.sch (EAGLE design)
At the start: 35 parts, among them J2 TC2030-CTX-NL, J3 IMPULSE_GECKO_HEADER, Q1 MOSFET-NCHANNELXFDN-3, U2 FM25LBTDFN-8, U3 NRF51822QF, X2 16MHz

Commit message: blast routed
Parts:
- removed J2: TC2030-CTX-NL, connector:TC2030-CTX-NL
- added C1: 0.8pF, passives:CAPACITOR
- added J1: TC2030-JLINK-NL, connector:TC2030-JLINK-NL
- L1: device SparkFun-Passives:INDUCTOR0603 -> passives:INDUCTOR0603; DIGIKEY 490-4025-1-ND -> (none)
- L2: value INDUCTOR0402 -> (none)
Connections:
- removed net !RESET: J2.!RESET
- removed net TCK: J2.TCK
- removed net TDO: J2.TDO
- removed net TMS: J2.TMS
- net !FRAM_CS: now also U3.P00/AREF0; no longer U3.P02/AIN3
- net !FRAM_HOLD: now also U3.P02/AIN3; no longer U3.P01/AIN2
- net !FRAM_WP: now also U3.P01/AIN2; no longer U3.P00/AREF0
- net GND: now also C1.2, J1.GND; no longer D1.C, D2.C, J2.GND
- net N$1: now also D2.C, U3.P15; no longer R2.1, U3.P10
- net N$11: now also C1.1
- net N$7: now also D1.C, U3.P10; no longer R1.1, U3.P09
- net SWDCLK: now also J1.SWDCLK
- net SWDIO: now also J1.SWDIO
- net VCC: now also J1.VCC, R1.1, R2.1; no longer J2.VCC
Other:
- moved on the sheet: A1, D1, D2, R1, R2

Commit message: update to bigger solar panel
- add footprint for big fram
- add footprint for rtc
Parts:
- removed R4, R5: 4.7k, passives:RESISTOR
- added C2: 0.1uF, passives:CAPACITOR
- added C4: 10nF, passives:CAPACITOR
- added R10, R11: 10k, passives:RESISTOR
- added R12, R9: 4.7k, passives:RESISTOR
- added U1: RV-3049-C3, chips:RV-3049-C3
- added U4: FM25V20-DG, chips:FM25V20-DG
- U3: DIGIKEY (none) -> 1490-1042-1-ND; MOUSER (none) -> 949-NRF51822-QFAC-R7
Connections:
- new net !FRAM2_CS: R9.1, U3.P24, U4.!CS
- new net BATTERY: C4.1, U1.VCC
- new net N$8: R10.2, U1.VBACKUP
- new net N$9: R11.2, U1.CLKOE
- new net RTC_CS: R12.2, U1.!CS, U3.P00/AREF0
- net !FRAM_CS: now also U3.P30; no longer U3.P00/AREF0
- net !FRAM_HOLD: no longer R4.1, U2.!HOLD
- net !FRAM_WP: no longer R5.1, U2.!WP
- net GND: now also C2.2, C4.2, R10.1, R11.1, R12.1, U1.GND, U4.VSS
- net MISO: now also U1.MISO, U4.SO
- net MOSI: now also U1.MOSI, U4.SI
- net N$7: now also U3.P14; no longer U3.P10
- net SCK: now also U1.SCL, U4.SCK
- net VCC: now also C2.1, R9.2, U2.!HOLD, U2.!WP, U4.!HOLD, U4.!WP, U4.VDD; no longer R4.2, R5.2
Other:
- note added: "FRAM"
- note added: "RTC"

Commit message: add blast files
Parts:
- removed C16: 2.2uF, passives:CAPACITOR
- removed J3: IMPULSE_GECKO_HEADER, gecko:IMPULSE_GECKO_HEADER
- removed R11: 10k, passives:RESISTOR
- removed R12: 4.7k, passives:RESISTOR
- added C14: 4.7uF, passives:CAPACITOR
- added J2: TC2030-JLINK-NL, connector:TC2030-JLINK-NL
- added R4, R5: 4.7k, passives:RESISTOR
- added SJ4: SOLDERJUMPERNO, SparkFun-Passives:SOLDERJUMPERNO
- A1: RICHARDSON_RFPD (none) -> FR05-S1-N-0001B
- C10, C11: value 1nF -> 0.1uF; DIGIKEY 490-1303-1-ND -> 445-4952-1-ND
- C12: value 47nF -> 1uF; DIGIKEY 445-1264-1-ND -> 1276-1513-1-ND
- C13: value 2.2nF -> 2.2uF; DIGIKEY 490-5419-1-ND -> 445-3882-1-ND
- C2: value 0.1uF -> 12pF; DIGIKEY (none) -> 490-6197-1-ND
- C3: value 1uF -> 12pF; DIGIKEY 1276-1513-1-ND -> 490-6197-1-ND
- C4: value 10nF -> 1nF; DIGIKEY (none) -> 490-1303-1-ND
- C5: value 0.1uF -> 1nF; DIGIKEY (none) -> 490-1303-1-ND
- C6: value 4.7uF -> 2.2nF; DIGIKEY 445-5947-1-ND -> 490-5419-1-ND
- C7: value 0.1uF -> 10nF; DIGIKEY 445-4952-1-ND -> 445-1260-1-ND
- C8: value 12pF -> 47nF; DIGIKEY 490-6197-1-ND -> 445-1264-1-ND
- C9: value 12pF -> 0.1uF; DIGIKEY 490-6197-1-ND -> 445-4952-1-ND
- D1, D2: DIGIKEY (none) -> 160-1837-1-ND
- J1: value TC2030-JLINK-NL -> IMPULSE_GECKO_HEADER; device connector:TC2030-JLINK-NL -> gecko:IMPULSE_GECKO_HEADER
- L1: DIGIKEY (none) -> 490-4025-1-ND
- L2: value (none) -> 15nH
- R10: value 10k -> 4.7M; DIGIKEY (none) -> 541-4.7MJCT-ND
- R3: DIGIKEY (none) -> RHM4.7KCECT-ND
- R6: value 1M -> 10k; DIGIKEY (none) -> RHM10KCECT-ND
- R7: value 4.7M -> 10k; DIGIKEY (none) -> RHM10KCECT-ND
- R9: value 4.7k -> 1M; DIGIKEY (none) -> RHM1.0MCECT-ND
- U1: value RV-3049-C3 -> NRF51822QF; device chips:RV-3049-C3 -> chips:NRF51822QF; DIGIKEY (none) -> 1490-1042-1-ND; MOUSER (none) -> 949-NRF51822-QFAC-R7
- U3: value NRF51822QF -> RV-3049-C3; device chips:NRF51822QF -> chips:RV-3049-C3; DIGIKEY 1490-1042-1-ND -> (none); MOUSER 949-NRF51822-QFAC-R7 -> (none); NEWARK (none) -> RV-3049-C3
- renumbered B2 to B1, X2 to X1
Connections:
- removed net !FRAM_HOLD: U3.P02/AIN3
- removed net !FRAM_WP: U3.P01/AIN2
- net !FRAM2_CS: now also R4.1, U1.P24; no longer R9.1, U3.P24
- net !FRAM_CS: now also U1.P30; no longer U3.P30
- net BATTERY: now also C7.1, SJ4.1, U3.VCC; no longer C4.1, U1.VCC
- net GND: now also C14.2, J2.GND, R5.1, R9.1; no longer C16.2, J3.GND, R11.1, R12.1
- net MISO: now also J1.MISO, U1.P28, U3.MISO; no longer J3.MISO, U1.MISO, U3.P28
- net MOSI: now also J1.MOSI/SDA, U1.P29, U3.MOSI; no longer J3.MOSI/SDA, U1.MOSI, U3.P29
- net N$1: now also U1.P15; no longer U3.P15
- net N$12: now also C12.1, C4.1, U1.AVDD; no longer C10.1, C3.1, U3.AVDD
- net N$13: now also U1.DCC; no longer U3.DCC
- net N$16: now also C2.1, U1.XC1; no longer C8.1, U3.XC1
- net N$17: now also C3.1, U1.XC2; no longer C9.1, U3.XC2
- net N$18: now also C5.1, U1.DEC1; no longer C11.1, U3.DEC1
- net N$19: now also C8.1, U1.DEC2; no longer C12.1, U3.DEC2
- net N$20: now also J1.TRIGGER/P2.1; no longer J3.TRIGGER/P2.1
- net N$21: now also J1.SHTDWN/P2.0; no longer J3.SHTDWN/P2.0
- net N$22: now also J1.OVRVLT/P1.7; no longer J3.OVRVLT/P1.7
- net N$5: now also U1.ANT1; no longer U3.ANT1
- net N$6: now also U1.ANT2; no longer U3.ANT2
- net N$7: now also U1.P14; no longer U3.P14
- net N$8: now also R7.2, U3.VBACKUP; no longer R10.2, U1.VBACKUP
- net N$9: now also R6.2, U3.CLKOE; no longer R11.2, U1.CLKOE
- net OV: now also U1.P05/AIN6; no longer U3.P05/AIN6
- net RTC_CS: now also R5.2, U1.P00/AREF0, U3.!CS; no longer R12.2, U1.!CS, U3.P00/AREF0
- net SCK: now also J1.SCL, U1.P25, U3.SCL; no longer J3.SCL, U1.SCL, U3.P25
- net SHDN: now also U1.P04/AIN5; no longer U3.P04/AIN5
- net SWDCLK: now also J2.SWDCLK, U1.SWDCLK; no longer J1.SWDCLK, U3.SWDCLK
- net SWDIO: now also J2.SWDIO, U1.SWDIO/!RESET; no longer J1.SWDIO, U3.SWDIO/!RESET
- net TIME_CTL: now also R9.2, U1.P07; no longer R6.2, U3.P07
- net TRIG: now also U1.P03/AIN4; no longer U3.P03/AIN4
- net VCAP: now also J1.VCAP, SJ4.2; no longer J3.VCAP
- net VCC: now also C10.1, C11.1, C14.1, C9.1, J1.VREG, J2.VCC, R4.2, U1.VDD; no longer C2.1, C5.1, C6.1, C7.1, J1.VCC, J3.VREG, R9.2, U3.VDD
- net VDD_PA: now also C6.1, U1.VDD_PA; no longer C13.1, U3.VDD_PA
- net VTIMER: now also C13.1, R10.2, U1.P06/AIN7/AREF1; no longer C16.1, R7.2, U3.P06/AIN7/AREF1
Other:
- note added: "FRAM (2 Mbit)"
- note added: "FRAM (4 Kbit)"
- note removed: "FRAM"
